File: STM32_BluetoothPill.kicad_sch (KiCad schematic)
At the start: 43 parts, among them IC1 MLPF-WB-01E3, J1 USB_A, J2 Conn_01x04, J3 Conn_01x16, J4 Conn_01x16, J5 RFShield_OnePiece, SW1 SW_Push, SW2 SW_Push, U1 USBLC6-2SC6, U2 STM32WB55CEU6TR, U3 LD3985M33R_SOT23, Y1 Crystal_Small, Y2 Crystal_Small

Commit message: pcb first try
Parts:
- AE1: footprint RF_Antenna:Texas_SWRA117D_2.4GHz_Right -> RF_Antenna:Texas_SWRA117D_2.4GHz_Left
- U2: footprint lib:QFN50P700X700X60-49N -> Package_DFN_QFN:QFN-48-1EP_7x7mm_P0.5mm_EP5.45x5.45mm
Changed lines of the file:
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@@
     (property "Reference" "U2" (id 0) (at 151.13 17.78 0))
     (property "Value" "STM32WB55CEU6TR" (id 1) (at 151.13 20.32 0))
-    (property "Footprint" "lib:QFN50P700X700X60-49N" (id 2) (at 138.43 76.2 0)
+    (property "Footprint" "Package_DFN_QFN:QFN-48-1EP_7x7mm_P0.5mm_EP5.45x5.45mm" (id 2) (at 138.43 76.2 0)
       (effects (font (size 1.27 1.27)) (justify left bottom) hide)
     )
@@
       (effects (font (size 1.27 1.27)) (justify right))
     )
-    (property "Footprint" "RF_Antenna:Texas_SWRA117D_2.4GHz_Right" (id 2) (at 133.35 134.62 0)
+    (property "Footprint" "RF_Antenna:Texas_SWRA117D_2.4GHz_Left" (id 2) (at 133.35 134.62 0)
       (effects (font (size 1.27 1.27)) hide)
     )
@@
     )
     (path "/61f290f2-e1eb-4f8a-b92c-38159b53d6bd"
-      (reference "AE1") (unit 1) (value "Antenna_Shield") (footprint "RF_Antenna:Texas_SWRA117D_2.4GHz_Right")
+      (reference "AE1") (unit 1) (value "Antenna_Shield") (footprint "RF_Antenna:Texas_SWRA117D_2.4GHz_Left")
     )
     (path "/86ca5ff7-caf9-44e0-8879-59882912f851"
@@
     )
     (path "/1a9756fb-2fe4-4729-82a6-8fc705d912bc"
-      (reference "U2") (unit 1) (value "STM32WB55CEU6TR") (footprint "lib:QFN50P700X700X60-49N")
+      (reference "U2") (unit 1) (value "STM32WB55CEU6TR") (footprint "Package_DFN_QFN:QFN-48-1EP_7x7mm_P0.5mm_EP5.45x5.45mm")
     )
     (path "/69eb8847-3a16-4dc2-b290-73e92782f93c"
